Commit message: mwe with gripper pads

File: franka_description/robots/franka_panda_fem_simple_v4_with_arm.urdf (robot description, URDF)
Before this commit: robot panda, 17 links, 16 joints
Links:
- added link panda_left_finger_pad
- added link panda_right_finger_pad
Joints:
- added joint left_finger_to_pad: type fixed, parent panda_left_finger_rigid, child panda_left_finger_pad, origin xyz=0.0 0.0 0.0 rpy=0.0 0.0 0.0
- added joint right_finger_to_pad: type fixed, parent panda_right_finger_rigid, child panda_right_finger_pad, origin xyz=0.0 0.0 0.0 rpy=0.0 0.0 0.0

Commit message: Perform pickup with Franka gripper on rigid object

File: franka_description/robots/franka_panda_fem_simple_v4_with_arm.urdf (robot description, URDF)
Before this commit: robot panda, 19 links, 18 joints
Joints:
- joint panda_left_finger_joint: limit lower=0.0 upper=0.04 effort=1e9 velocity=1e9 -> lower=0.0 upper=0.04 effort=1e2 velocity=1e2
- joint panda_right_finger_joint: limit lower=0.0 upper=0.04 effort=1e9 velocity=1e9 -> lower=0.0 upper=0.04 effort=1e2 velocity=1e2
