Commit message: work with example rect obj

File: examples/rectangle/rectangle.urdf (robot description, URDF)
Before this commit: robot root, 1 links, 0 joints
Links:
- removed link link_rectangle_convex_piece_0
- added link link_rectangle, mass 3.45E-05; collision mesh filename=rectangle.obj scale=1.0000E+00 1.0000E+00 1.0000E+00; visual mesh filename=rectangle.obj scale=1.0000E+00 1.0000E+00 1.0000E+00
