Commit message: Add finger pads, but they are not positioned correctly yet.

File: yumi_description/urdf/yumi.urdf (robot description, URDF)
Before this commit: robot yumi, 12 links, 11 joints
Links:
- added link right_finger_pad
Joints:
- added joint right_finger_to_pad: type fixed, parent gripper_r_finger_r, child right_finger_pad, origin xyz=0.0 0.0 0.0 rpy=0.0 0.0 0.0

Commit message: Change limits of Yumi gripper so they can open even wider

File: yumi_description/urdf/yumi.urdf (robot description, URDF)
Before this commit: robot yumi, 13 links, 12 joints
Joints:
- joint gripper_r_joint: limit lower=-0.025 upper=0 effort=20 velocity=2 -> lower=-0.025 upper=0.02 effort=20 velocity=2
- joint gripper_r_joint_m: limit lower=-0.025 upper=0 effort=20 velocity=2 -> lower=-0.025 upper=0.02 effort=20 velocity=2
